File: mpu-9150_breakout/mpu-9150_breakout.kicad_pcb (KiCad board)
At the start: 2 copper layers, 15.2 x 12.7 mm, 11 parts, among them P1 CONN_1, P2 CONN_5, P3 CONN_5, U1 MPU-9150

Commit message: Add missing file
Parts:
- GS1, GS2, GS3: moved to B.Cu
- moved C4 3.94 mm to (351.2, 210.1), turned to 180 degrees
- moved P1 2.54 mm to (345.4, 200.7)
- moved C1 0.85 mm to (351.2, 208.7)
- moved C2 0.52 mm to (352.4, 205.2)
- moved C3 0.38 mm to (350.6, 201.7)
- turned GS1 to 270 degrees
- turned GS2 to 90 degrees
- turned GS3 to 270 degrees
Routing:
- net GND: track 49.3 -> 42.9 mm, vias 2 -> 1
- net /CLKOUT: track 2.69 -> 4.78 mm
- net /INT: track 6.52 -> 5.74 mm
- net /ES_CL: track 7.61 -> 6.86 mm
- net VDD: track 21.2 -> 20.5 mm, vias 1 -> 2
- net /FSYNC: track 9.63 -> 10.2 mm
- net /CLKIN: track 12.7 -> 12.4 mm, vias 2 -> 1
- net /AD0: vias 0 -> 1
Other:
- board text added: "11 10 9 8 7"
- board text added: "1|2 3 4 5 6"
- board text added: "IMU"
- board text added: "Invensense MPU-9150"
- board text added: "X"
- board text added: "Y"
- board text added: "Z"

Commit message: Adding pin names to silk screen
Other:
- board text added: "CLK OUT"
- board text added: "CLKIN"
- board text added: "ESCL"
- board text added: "ESDA"
- board text added: "FSYNC"
- board text added: "GND"
- board text added: "INT"
- board text added: "SCL"
- board text added: "SDA"
- board text added: "VDD"
- board text added: "VLOG"
- board text removed: "11 10 9 8 7"
- board text removed: "1|2 3 4 5 6"
Changed lines of the file:
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@@
     (links 29)
     (no_connects 0)
-    (area 341.579999 199.339999 356.920001 212.140001)
+    (area 338.455 196.3766 360.172 214.5954)
     (thickness 1.6)
-    (drawings 48)
+    (drawings 57)
     (tracks 105)
     (zones 0)
@@
   (layers
     (15 F.Cu signal)
-    (0 B.Cu signal)
+    (0 B.Cu signal hide)
     (16 B.Adhes user hide)
     (17 F.Adhes user hide)
@@
     )
   )
+  (gr_text "CLK\nOUT" (at 347.6752 200.6346 270) (layer B.SilkS)
+    (effects (font (size 0.6 0.6) (thickness 0.05)) (justify mirror))
+  )
+  (gr_text ESCL (at 344.17 210.82 270) (layer B.SilkS)
+    (effects (font (size 0.6 0.6) (thickness 0.05)) (justify mirror))
+  )
+  (gr_text ESDA (at 344.17 208.28 270) (layer B.SilkS)
+    (effects (font (size 0.6 0.6) (thickness 0.05)) (justify mirror))
+  )
+  (gr_text CLKIN (at 344.17 205.74 270) (layer B.SilkS)
+    (effects (font (size 0.6 0.6) (thickness 0.05)) (justify mirror))
+  )
+  (gr_text SDA (at 344.17 203.2 270) (layer B.SilkS)
+    (effects (font (size 0.6 0.6) (thickness 0.05)) (justify mirror))
+  )
+  (gr_text SCL (at 344.17 200.66 270) (layer B.SilkS)
+    (effects (font (size 0.6 0.6) (thickness 0.05)) (justify mirror))
+  )
+  (gr_text VLOG (at 354.33 210.82 270) (layer B.SilkS)
+    (effects (font (size 0.6 0.6) (thickness 0.05)) (justify mirror))
+  )
+  (gr_text FSYNC (at 354.33 208.28 270) (layer B.SilkS)
+    (effects (font (size 0.6 0.6) (thickness 0.05)) (justify mirror))
+  )
+  (gr_text INT (at 354.33 205.74 270) (layer B.SilkS)
+    (effects (font (size 0.6 0.6) (thickness 0.05)) (justify mirror))
+  )
+  (gr_text VDD (at 354.33 203.2 270) (layer B.SilkS)
+    (effects (font (size 0.6 0.6) (thickness 0.05)) (justify mirror))
+  )
+  (gr_text GND (at 354.33 200.66 270) (layer B.SilkS)
+    (effects (font (size 0.6 0.6) (thickness 0.05)) (justify mirror))
+  )
   (gr_text IMU (at 350.393 203.835) (layer B.SilkS)
     (effects (font (size 1.5 1.5) (thickness 0.3)) (justify mirror))
   )
-  (gr_text "Invensense\nMPU-9150\n" (at 350.647 200.152) (layer B.SilkS)
-    (effects (font (size 0.762 0.762) (thickness 0.127)) (justify mirror))
+  (gr_text "Invensense\nMPU-9150\n" (at 351.155 200.025) (layer B.SilkS)
+    (effects (font (size 0.6 0.6) (thickness 0.127)) (justify mirror))
   )
   (gr_text Z (at 348.615 206.629) (layer B.SilkS)
     (effects (font (size 1.5 1.5) (thickness 0.3) italic) (justify mirror))
   )
-  (gr_text Y (at 346.837 202.565) (layer B.SilkS)
+  (gr_text Y (at 346.075 203.2) (layer B.SilkS)
     (effects (font (size 1.5 1.5) (thickness 0.3) italic) (justify mirror))
   )
@@
   (gr_line (start 346.837 207.01) (end 346.837 204.724) (angle 90) (layer B.SilkS) (width 0.2))
   (gr_circle (center 346.837 208.026) (end 346.837 207.01) (layer B.SilkS) (width 0.2))
-  (gr_text "11\n10\n9\n8\n7" (at 354.076 203.327) (layer B.SilkS)
-    (effects (font (size 0.762 0.762) (thickness 0.1905)) (justify left mirror))
-  )
-  (gr_text "1|2\n3\n4\n5\n6" (at 344.297 203.2) (layer B.SilkS)
-    (effects (font (size 0.762 0.762) (thickness 0.1905)) (justify right mirror))
-  )
   (gr_line (start 341.63 199.39) (end 341.63 212.09) (angle 90) (layer Edge.Cuts) (width 0.1))
   (gr_line (start 356.87 199.39) (end 341.63 199.39) (angle 90) (layer Edge.Cuts) (width 0.1))
