File: flyingf3_shield/flyingf3_shield.sch (KiCad schematic (older format))
At the start: 1 part

Commit message: pushing current local state
Parts:
- removed uC?: STM32F3, ~, symbol STM32F3
- added DISCO1: STM32F3DISCOVERY, ~, symbol STM32F3DISCOVERY
- added PWM1: PWM_IN8, symbol PWM_IN8
- added PWM2: PWM_OUT10, symbol PWM_OUT10
Connections:
- net PWM_IN_1: now also DISCO1.67 (PA8), PWM1.3 (Signal1)
- net PWM_IN_2: now also DISCO1.95 (PB8), PWM1.4 (Signal2)
- net PWM_IN_3: now also DISCO1.96 (PB9), PWM1.5 (Signal3)
- net PWM_IN_4: now also DISCO1.63 (PC6), PWM1.6 (Signal4)
- net PWM_IN_5: now also DISCO1.64 (PC7), PWM1.7 (Signal5)
- net PWM_IN_6: now also DISCO1.65 (PC8), PWM1.8 (Signal6)
- net PWM_IN_7: now also DISCO1.10 (PF9), PWM1.9 (Signal7)
- net PWM_IN_8: now also DISCO1.11 (PF10), PWM1.10 (Signal8)
- net PWM_OUT_1: now also DISCO1.59 (PD12), PWM2.3 (Signal1)
- net PWM_OUT_10: now also DISCO1.29 (PA4), PWM2.12 (Signal10)
- net PWM_OUT_2: now also DISCO1.60 (PD13), PWM2.4 (Signal2)
- net PWM_OUT_3: now also DISCO1.61 (PD14), PWM2.5 (Signal3)
- net PWM_OUT_4: now also DISCO1.62 (PD15), PWM2.6 (Signal4)
- net PWM_OUT_5: now also DISCO1.24 (PA1), PWM2.7 (Signal5)
- net PWM_OUT_6: now also DISCO1.25 (PA2), PWM2.8 (Signal6)
- net PWM_OUT_7: now also DISCO1.26 (PA3), PWM2.9 (Signal7)
- net PWM_OUT_8: now also DISCO1.35 (PB0), PWM2.10 (Signal8)
- net PWM_OUT_9: now also DISCO1.36 (PB1), PWM2.11 (Signal9)
- new net CAN_RX: DISCO1.81 (PD0)
- new net CAN_TX: DISCO1.82 (PD1)
- new net EXT_INT_1: DISCO1.5 (PE6)
- new net EXT_INT_2: DISCO1.84 (PD3)
- new net EXT_INT_3: DISCO1.85 (PD4)
- new net EXT_INT_4: DISCO1.88 (PD7)
- new net GND: DISCO1.49 (GND), DISCO1.50 (GND), DISCO1.74 (GND), DISCO1.75 (GND), DISCO1.99 (GND), PWM1.1 (GND), PWM2.1 (GND)
- new net SPI3_CS2: DISCO1.47 (PB10)
- new net SPI3_CS3: DISCO1.48 (PB11)
- new net SPI3_CS4: DISCO1.51 (PB12)
- new net SPI3_CS5: DISCO1.52 (PB13)
- new net SPI3_MISO: DISCO1.90 (PB4)
- new net SPI3_MOSI: DISCO1.91 (PB5)
- new net SPI3_NSS: DISCO1.77 (PA15)
- new net SPI3_SCK: DISCO1.89 (PB3)
- new net UART4_RX: DISCO1.79 (PC11)
- new net UART4_TX: DISCO1.78 (PC10)
- new net UART5_RX: DISCO1.83 (PD2)
- new net UART5_TX: DISCO1.80 (PC12)
- new net USART1_RX: DISCO1.68 (PA9)
- new net USART1_TX: DISCO1.34 (PC5)
- new net USART2_RX: DISCO1.87 (PD6)
- new net USART2_TX: DISCO1.86 (PD5)
- new net USART3_RX: DISCO1.56 (PD9)
- new net USART3_TX: DISCO1.55 (PD8)
- new net VCC_3V: DISCO1.20 (VCC_3V), DISCO1.6 (VCC_3V)
- new net VCC_5V: DISCO1.21 (VCC_5V), DISCO1.22 (VCC_5V)
- new net VDD: DISCO1.28 (VDD)
Changed lines of the file:
@@
 LIBS:valves
 LIBS:stmicro
+LIBS:pwm
+LIBS:ab2_header
+LIBS:flyingf3_shield-cache
 EELAYER 27 0
 EELAYER END
@@
 Sheet 1 1
 Title ""
-Date "12 feb 2014"
+Date "13 feb 2014"
 Rev ""
 Comp ""
@@
 Comment4 ""
 $EndDescr
+Text Label 2900 1350 0    60   ~ 0
+GND
+Text Label 2900 1450 0    60   ~ 0
+GND
+Text Label 2900 1550 0    60   ~ 0
+GND
+Text Label 2900 1650 0    60   ~ 0
+GND
+Text Label 2900 1750 0    60   ~ 0
+GND
+Text Label 1500 1350 2    60   ~ 0
+VCC_3V
+Text Label 1500 1450 2    60   ~ 0
+VCC_3V
+Text Label 1500 1600 2    60   ~ 0
+VCC_5V
+Text Label 1500 1700 2    60   ~ 0
+VCC_5V
+Text Label 1500 1850 2    60   ~ 0
+VDD
 $Comp
-L STM32F3 uC?
-U 1 1 52FB115D
-P 6100 3850
-F 0 "uC?" H 6100 1300 60  0000 C CNN
-F 1 "STM32F3" H 6100 6400 60  0000 C CNN
-F 2 "~" H 7950 1100 60  0000 C CNN
-F 3 "~" H 7950 1100 60  0000 C CNN
-	1    6100 3850
+L STM32F3DISCOVERY DISCO1
+U 1 1 52FC4DC1
+P 2200 4150
+F 0 "DISCO1" H 2200 1250 60  0000 C CNN
+F 1 "STM32F3DISCOVERY" H 2200 7200 60  0000 C CNN
+F 2 "~" H 3200 1050 60  0000 C CNN
+F 3 "~" H 3200 1050 60  0000 C CNN
+	1    2200 4150
 	1    0    0    -1
 $EndComp
-Text Label 5500 2250 2    60   ~ 0
+Text Label 1100 2900 2    60   ~ 0
 PWM_IN_1
-Text Label 5500 3900 2    60   ~ 0
+Text Label 3300 2900 0    60   ~ 0
 PWM_IN_2
-Text Label 5500 4000 2    60   ~ 0
+Text Label 3300 3000 0    60   ~ 0
 PWM_IN_3
-Text Label 6700 2350 0    60   ~ 0
+Text Label 1100 4350 2    60   ~ 0
 PWM_IN_4
-Text Label 6700 2250 0    60   ~ 0
+Text Label 1100 4450 2    60   ~ 0
 PWM_IN_5
-Text Label 6700 2150 0    60   ~ 0
+Text Label 1100 4550 2    60   ~ 0
 PWM_IN_6
-Text Label 5500 5250 2    60   ~ 0
+Text Label 3300 6300 0    60   ~ 0
 PWM_IN_7
-Text Label 5500 5350 2    60   ~ 0
+Text Label 3300 6400 0    60   ~ 0
 PWM_IN_8
-Text Label 6700 3400 0    60   ~ 0
+Text Label 3300 4950 0    60   ~ 0
 PWM_OUT_1
-Text Label 6700 3300 0    60   ~ 0
+Text Label 3300 5050 0    60   ~ 0
 PWM_OUT_2
-Text Label 6700 3200 0    60   ~ 0
+Text Label 3300 5150 0    60   ~ 0
 PWM_OUT_3
-Text Label 6700 3100 0    60   ~ 0
+Text Label 3300 5250 0    60   ~ 0
 PWM_OUT_4
-Text Label 5500 1550 2    60   ~ 0
+Text Label 1100 2200 2    60   ~ 0
 PWM_OUT_5
-Text Label 5500 1650 2    60   ~ 0
+Text Label 1100 2300 2    60   ~ 0
 PWM_OUT_6
-Text Label 5500 1750 2    60   ~ 0
+Text Label 1100 2400 2    60   ~ 0
 PWM_OUT_7
-Text Label 5500 3100 2    60   ~ 0
+Text Label 3300 2100 0    60   ~ 0
 PWM_OUT_8
-Text Label 5500 3200 2    60   ~ 0
+Text Label 3300 2200 0    60   ~ 0
 PWM_OUT_9
-Text Label 5500 1850 2    60   ~ 0
+Text Label 1100 2500 2    60   ~ 0
+PWM_OUT_10
+Text Label 1100 4250 2    60   ~ 0
+USART1_TX
+Text Label 3300 4250 0    60   ~ 0
+USART2_TX
+Text Label 3300 4550 0    60   ~ 0
+USART3_TX
+Text Label 1100 4750 2    60   ~ 0
+UART4_TX
+Text Label 1100 4950 2    60   ~ 0
+UART5_TX
+Text Label 1100 3000 2    60   ~ 0
+USART1_RX
+Text Label 3300 4350 0    60   ~ 0
+USART2_RX
+Text Label 3300 4650 0    60   ~ 0
+USART3_RX
+Text Label 1100 4850 2    60   ~ 0
+UART4_RX
+Text Label 3300 3950 0    60   ~ 0
+UART5_RX
+Text Label 3300 2400 0    60   ~ 0
+SPI3_SCK
+Text Label 3300 2500 0    60   ~ 0
+SPI3_MISO
+Text Label 3300 2600 0    60   ~ 0
+SPI3_MOSI
+Text Label 1100 3600 2    60   ~ 0
+SPI3_NSS
+Text Label 3300 3100 0    60   ~ 0
+SPI3_CS2
+Text Label 3300 3200 0    60   ~ 0
+SPI3_CS3
+Text Label 3300 3300 0    60   ~ 0
+SPI3_CS4
+Text Label 3300 3400 0    60   ~ 0
+SPI3_CS5
+Text Label 1100 6000 2    60   ~ 0
+EXT_INT_1
+Text Label 3300 4050 0    60   ~ 0
+EXT_INT_2
+Text Label 3300 4150 0    60   ~ 0
+EXT_INT_3
+Text Label 3300 4450 0    60   ~ 0
+EXT_INT_4
+Text Label 3300 3750 0    60   ~ 0
+CAN_RX
+Text Label 3300 3850 0    60   ~ 0
+CAN_TX
+$Comp
+L PWM_IN8 PWM1
+U 1 1 52FD11DA
+P 5600 2200
+F 0 "PWM1" H 5600 1250 60  0000 C CNN
+F 1 "PWM_IN8" H 5600 2450 60  0000 C CNN
+F 2 "" H 5600 2450 60  0000 C CNN
+F 3 "" H 5600 2450 60  0000 C CNN
+	1    5600 2200
+	1    0    0    -1
+$EndComp
+$Comp
+L PWM_OUT10 PWM2
+U 1 1 52FD11FD
+P 5600 3600
+F 0 "PWM2" H 5600 2450 60  0000 C CNN
+F 1 "PWM_OUT10" H 5600 3850 60  0000 C CNN
+F 2 "" H 5600 3850 60  0000 C CNN
+F 3 "" H 5600 3850 60  0000 C CNN
+	1    5600 3600
+	1    0    0    -1
+$EndComp
+Text Label 5100 2100 2    60   ~ 0
+GND
+Text Label 5100 3500 2    60   ~ 0
+GND
+Text Label 5100 2300 2    60   ~ 0
+PWM_IN_1
+Text Label 5100 2400 2    60   ~ 0
+PWM_IN_2
+Text Label 5100 2500 2    60   ~ 0
+PWM_IN_3
+Text Label 5100 2600 2    60   ~ 0
+PWM_IN_4
+Text Label 5100 2700 2    60   ~ 0
+PWM_IN_5
+Text Label 5100 2800 2    60   ~ 0
+PWM_IN_6
+Text Label 5100 2900 2    60   ~ 0
+PWM_IN_7
+Text Label 5100 3000 2    60   ~ 0
+PWM_IN_8
+Text Label 5100 3700 2    60   ~ 0
+PWM_OUT_1
+Text Label 5100 3800 2    60   ~ 0
+PWM_OUT_2
+Text Label 5100 3900 2    60   ~ 0
+PWM_OUT_3
+Text Label 5100 4000 2    60   ~ 0
+PWM_OUT_4
+Text Label 5100 4100 2    60   ~ 0
+PWM_OUT_5
+Text Label 5100 4200 2    60   ~ 0
+PWM_OUT_6
+Text Label 5100 4300 2    60   ~ 0
+PWM_OUT_7
+Text Label 5100 4400 2    60   ~ 0
+PWM_OUT_8
+Text Label 5100 4500 2    60   ~ 0
+PWM_OUT_9
+Text Label 5100 4600 2    60   ~ 0
 PWM_OUT_10
 $EndSCHEMATC
