File: ms5611_breakout/ms5611_breakout.kicad_pcb (KiCad board)
At the start: 2 copper layers, 7 parts, among them P1 CONN_4, P2 CONN_4

Commit message: Finish first version of the breakout board.
Parts:
- removed ms5611 (x2): VAL**, ms5611
- added U1: MS5611, ms5611, B.Cu at (351.5, 235.8)
- P1, P2: moved to B.Cu
- moved GS2 5.06 mm to (352.6, 235.2)
- moved C1 1.08 mm to (355.1, 235.2)
- moved GS1 0.81 mm to (352.6, 239.4), turned to 180 degrees
Routing:
- net /VDD: track 0.00 -> 18.8 mm, vias 0 -> 1
- net /CSB: track 0.00 -> 14.5 mm, vias 0 -> 1
- net /GND: track 0.00 -> 13.4 mm, vias 0 -> 1
- net /SDO: track 0.00 -> 3.30 mm
- net /SDI/SDA: track 0.00 -> 2.77 mm
- net /SCLK: track 0.00 -> 2.68 mm
- net /PS: track 4.63 -> 7.25 mm, vias 0 -> 1
- added copper zone on F.Cu, net /GND
Other:
- board outline added: 12.7 x 10.2 mm
- net class Default: clearance 0.254 -> 0.1524; via_dia 0.889 -> 0.6858; via_drill 0.635 -> 0.3302
- net class OSH Min added: clearance 0.1524, trace_width 0.1524, via_dia 0.6858, via_drill 0.3302
- net class POWER added: clearance 0.2032, trace_width 0.381, via_dia 0.889, via_drill 0.3302
- rule trace_clearance: 0.254 -> 0.1524
- rule trace_min: 0.254 -> 0.1524
- rule via_min_drill: 0.508 -> 0.3302
- rule via_min_size: 0.889 -> 0.6858
- board text added: "0xEC"
- board text added: "0xEE"
- board text added: "CSB"
- board text added: "GND"
- board text added: "I2C"
- board text added: "I²C Address"
- board text added: "MS5611-01BA03"
- board text added: "PS"
- board text added: "Protocol"
- board text added: "SCLK"
- board text added: "SDA/I"
- board text added: "SDO"
- board text added: "SPI"
- board text added: "VDD"
